Commit message: Add Farmily RB5 robot model

File: ros2_ws/src/rbpodo_ros2/rbpodo_description/robots/rb5_850e.urdf.xacro (robot description, xacro)
@@ -16,28 +16,4 @@
   <xacro:property name="wrist3_tc" value="${1}" />
   <xacro:rb_6dof model_id="rb5_850e" prefix="$(arg prefix)" tcp_name="tcp" tcp_xyz="0 -0.0967 0" tcp_rpy="0 0 0" />
-  <!-- Tomato gripper CAD is authored in millimetres with its mounting frame
-       at the RB5 flange origin. Keep tcp as the MoveIt planning tip. -->
-  <link name="$(arg prefix)tomato_gripper">
-    <visual>
-      <geometry>
-        <mesh filename="package://rbpodo_description/meshes/tomato_gripper/tomato_gripper.stl"
-              scale="0.001 0.001 0.001" />
-      </geometry>
-      <material name="tomato_gripper_gray">
-        <color rgba="0.25 0.25 0.28 1.0" />
-      </material>
-    </visual>
-    <collision>
-      <geometry>
-        <mesh filename="package://rbpodo_description/meshes/tomato_gripper/tomato_gripper.stl"
-              scale="0.001 0.001 0.001" />
-      </geometry>
-    </collision>
-  </link>
-  <joint name="$(arg prefix)tomato_gripper_joint" type="fixed">
-    <origin xyz="0 0 0" rpy="0 0 0" />
-    <parent link="$(arg prefix)link6" />
-    <child link="$(arg prefix)tomato_gripper" />
-  </joint>
   <xacro:rb_6dof_ros2_control prefix="$(arg prefix)" robot_ip="$(arg robot_ip)" cb_simulation="$(arg cb_simulation)" use_fake_hardware="$(arg use_fake_hardware)" fake_sensor_commands="$(arg fake_sensor_commands)" torque_constants="${[base_tc, shoulder_tc, elbow_tc, wrist1_tc, wrist2_tc, wrist3_tc]}" />
 </robot>

File: ros2_ws/src/rbpodo_ros2/rbpodo_moveit_config/config/rbpodo.urdf.xacro (robot description, xacro)
@@ -1,5 +1,5 @@
 <?xml version="1.0"?>
 <robot xmlns:xacro="http://www.ros.org/wiki/xacro" name="rb">
-    <xacro:arg name="model_id" default="rb5_850e" />
+    <xacro:arg name="model_id" default="rb5_farmily" />
     <!--robot name="$(arg model_id)"/-->
     <!-- Import rb urdf file -->
