Commit message: 수확 계획 비교 기능과 작업 공간 안전 설정 확장
- Cartesian, OMPL, CHOMP, PILZ LIN pre-grasp 플래너 선택과 지속 Planner 실행을 연결

- fake hardware를 PICK_READY 관절 자세로 초기화하고 실제 로봇 상태와 분리

- OMPL 관절 제약을 각 단계 시작 자세 중심 ±120도로 적용하되 wrist3는 제외

- Plan 성공과 실패 모두에서 현재 자세부터 pre-grasp까지 관절 최소·최대·변화폭을 GUI 로그와 결과 데이터에 기록

- 작업 공간 좌우 가벽, 천장과 로봇 받침대 collision 및 실행 스크립트 치수 옵션 추가

- CHOMP용 PILZ endpoint seed와 Cartesian 복귀 fallback을 추가하고 관련 테스트 및 문서 갱신

File: ros2_ws/src/rbpodo_ros2/rbpodo_description/robots/rb_6dof.ros2_control.xacro (robot description, xacro)
@@ -1,5 +1,11 @@
 <?xml version='1.0' encoding='utf-8'?>
 <robot xmlns:xacro="http://www.ros.org/wiki/xacro">
-  <xacro:macro name="rb_6dof_ros2_control" params="prefix robot_ip cb_simulation:=^|false use_fake_hardware:=^|false fake_sensor_commands:=^|false torque_constants:=${[1, 1, 1, 1, 1, 1]}">
+  <xacro:arg name="initial_base" default="0.0"/>
+  <xacro:arg name="initial_shoulder" default="0.0"/>
+  <xacro:arg name="initial_elbow" default="0.0"/>
+  <xacro:arg name="initial_wrist1" default="0.0"/>
+  <xacro:arg name="initial_wrist2" default="0.0"/>
+  <xacro:arg name="initial_wrist3" default="0.0"/>
+  <xacro:macro name="rb_6dof_ros2_control" params="prefix robot_ip cb_simulation:=^|false use_fake_hardware:=^|false fake_sensor_commands:=^|false torque_constants:=${[1, 1, 1, 1, 1, 1]} initial_positions:=${[float('$(arg initial_base)'), float('$(arg initial_shoulder)'), float('$(arg initial_elbow)'), float('$(arg initial_wrist1)'), float('$(arg initial_wrist2)'), float('$(arg initial_wrist3)')]}">
     <ros2_control name="RBPodoHardwareInterface" type="system">
       <hardware>
@@ -15,21 +21,24 @@
         </xacro:unless>
       </hardware>
-      <xacro:macro name="configure_joint" params="joint_name torque_constant:=1">
+      <xacro:macro name="configure_joint" params="joint_name torque_constant:=1 initial_position:=0">
         <joint name="${joint_name}">
-          <param name="initial_position">0.0</param>
           <param name="torque_constant">${torque_constant}</param>
           <command_interface name="effort"/>
           <command_interface name="velocity"/>
           <command_interface name="position"/>
-          <state_interface name="position"/>
-          <state_interface name="effort"/>
+          <state_interface name="position">
+            <param name="initial_value">${initial_position}</param>
+          </state_interface>
+          <state_interface name="effort">
+            <param name="initial_value">0.0</param>
+          </state_interface>
         </joint>
       </xacro:macro>
-      <xacro:configure_joint joint_name="${prefix}base" torque_constant="${torque_constants[0]}" />
-      <xacro:configure_joint joint_name="${prefix}shoulder" torque_constant="${torque_constants[1]}" />
-      <xacro:configure_joint joint_name="${prefix}elbow" torque_constant="${torque_constants[2]}" />
-      <xacro:configure_joint joint_name="${prefix}wrist1" torque_constant="${torque_constants[3]}" />
-      <xacro:configure_joint joint_name="${prefix}wrist2" torque_constant="${torque_constants[4]}" />
-      <xacro:configure_joint joint_name="${prefix}wrist3" torque_constant="${torque_constants[5]}" />
+      <xacro:configure_joint joint_name="${prefix}base" torque_constant="${torque_constants[0]}" initial_position="${initial_positions[0]}" />
+      <xacro:configure_joint joint_name="${prefix}shoulder" torque_constant="${torque_constants[1]}" initial_position="${initial_positions[1]}" />
+      <xacro:configure_joint joint_name="${prefix}elbow" torque_constant="${torque_constants[2]}" initial_position="${initial_positions[2]}" />
+      <xacro:configure_joint joint_name="${prefix}wrist1" torque_constant="${torque_constants[3]}" initial_position="${initial_positions[3]}" />
+      <xacro:configure_joint joint_name="${prefix}wrist2" torque_constant="${torque_constants[4]}" initial_position="${initial_positions[4]}" />
+      <xacro:configure_joint joint_name="${prefix}wrist3" torque_constant="${torque_constants[5]}" initial_position="${initial_positions[5]}" />
     </ros2_control>
   </xacro:macro>
