Commit message: Add tomato scene and gripper planning tip

File: ros2_ws/src/rbpodo_ros2/rbpodo_description/robots/rb5_farmily.urdf.xacro (robot description, xacro)
@@ -29,3 +29,15 @@
     <child link="$(arg prefix)tomato_gripper" />
   </joint>
+  <!--
+    Planning TCP at the distal center of the tomato gripper. The STL is in
+    millimetres and extends to x=-211.6 mm; y=10.75 mm is the center of the
+    rounded tip at that section. Keep this fixed joint separate so the TCP can
+    be calibrated without moving the visual/collision mesh.
+  -->
+  <link name="$(arg prefix)tomato_gripper_tip" />
+  <joint name="$(arg prefix)tomato_gripper_tip_joint" type="fixed">
+    <origin xyz="-0.2116 0.01075 0" rpy="0 0 0" />
+    <parent link="$(arg prefix)tomato_gripper" />
+    <child link="$(arg prefix)tomato_gripper_tip" />
+  </joint>
 </robot>

Commit message: RealSense D435 모델 및 수확 도구 좌표계 통합
공식 RealSense D435 시각 메시와 nominal depth/color/infrared 프레임, 단순화된 충돌 형상, 원본 출처 및 라이선스를 추가했다. 토마토 그리퍼에 D435를 장착하고 위치와 회전을 Xacro 인자로 조정할 수 있도록 구성했으며, 사용자가 보정한 카메라 장착값과 tomato_gripper_tip RPY를 로봇 모델에 반영했다. RViz에서도 새 카메라 링크와 optical TF를 확인할 수 있도록 표시 구성을 저장했다.

Cartesian 수확 코드가 tomato_gripper에서 tomato_gripper_tip까지의 고정 회전을 TF에서 읽어 목표 자세에 자동 합성하도록 수정했다. 따라서 이후 tip RPY를 다시 보정해도 수확 자세 계산에 회전값을 하드코딩할 필요가 없다. 계획 경로가 RViz에서 누락되지 않도록 DisplayTrajectory의 로봇 모델 ID를 수정하고, tip 고정 회전 합성을 검증하는 회귀 테스트와 토마토 회전 보조 스크립트도 추가했다.

check_urdf와 DAE XML 검증, 수확 기하 단위 테스트 3개, 관련 ROS 2 패키지 빌드, fake-hardware MoveIt 기동을 확인했다. 변경된 tip RPY가 적용된 plan-only 수확 시험에서도 토마토-그리퍼-줄기 배치 조건을 통과했고 Cartesian 경로 fraction 1.000을 확인했다.

File: ros2_ws/src/rbpodo_ros2/rbpodo_description/robots/rb5_farmily.urdf.xacro (robot description, xacro)
@@ -3,4 +3,11 @@
   <!-- Keep the Rainbow Robotics RB5 model as the unmodified base robot. -->
   <xacro:include filename="$(find rbpodo_description)/robots/rb5_850e.urdf.xacro" />
+  <xacro:include filename="$(find rbpodo_description)/robots/realsense_d435.urdf.xacro" />
+  <xacro:arg name="d435_mount_x" default="-0.11" />
+  <xacro:arg name="d435_mount_y" default="-0.10" />
+  <xacro:arg name="d435_mount_z" default="0.0" />
+  <xacro:arg name="d435_mount_roll" default="-1.57" />
+  <xacro:arg name="d435_mount_pitch" default="0.0" />
+  <xacro:arg name="d435_mount_yaw" default="3.141592" />
   <!-- Farmily-specific links and joints belong below this line. -->
   <link name="$(arg prefix)tomato_gripper">
@@ -37,7 +44,20 @@
   <link name="$(arg prefix)tomato_gripper_tip" />
   <joint name="$(arg prefix)tomato_gripper_tip_joint" type="fixed">
-    <origin xyz="-0.2116 0.01075 0" rpy="0 0 0" />
+    <origin xyz="-0.2116 0.01075 0" rpy="1.57 3.14 0" />
     <parent link="$(arg prefix)tomato_gripper" />
     <child link="$(arg prefix)tomato_gripper_tip" />
   </joint>
+  <!--
+    D435 mounted above the gripper with its optical axis facing the gripper
+    tip. These six mount arguments are calibration values and can be adjusted
+    without editing the reusable camera model.
+  -->
+  <xacro:realsense_d435
+    parent="$(arg prefix)tomato_gripper"
+    name="$(arg prefix)d435"
+    use_mesh="true">
+    <origin
+      xyz="$(arg d435_mount_x) $(arg d435_mount_y) $(arg d435_mount_z)"
+      rpy="$(arg d435_mount_roll) $(arg d435_mount_pitch) $(arg d435_mount_yaw)" />
+  </xacro:realsense_d435>
 </robot>

Commit message: RB5 베이스에 Farmily 리프트 어셈블리 연결
Assy_Lift STL 메시를 rbpodo_description 패키지 리소스로 추가한다.\n\n리프트 링크를 link0의 fixed child로 구성하고 위치 및 회전 조정용 Xacro 인자를 제공한다. 조정된 기본 장착 좌표와 밀리미터 단위 메시 스케일을 반영한다.

File: ros2_ws/src/rbpodo_ros2/rbpodo_description/robots/rb5_farmily.urdf.xacro (robot description, xacro)
@@ -10,5 +10,32 @@
   <xacro:arg name="d435_mount_pitch" default="0.0" />
   <xacro:arg name="d435_mount_yaw" default="3.141592" />
+  <!-- Farmily lift pose relative to the RB5 base frame (link0). -->
+  <xacro:arg name="lift_mount_x" default="0.0" />
+  <xacro:arg name="lift_mount_y" default="0.6" />
+  <xacro:arg name="lift_mount_z" default="-0.35" />
+  <xacro:arg name="lift_mount_roll" default="1.57" />
+  <xacro:arg name="lift_mount_pitch" default="0.0" />
+  <xacro:arg name="lift_mount_yaw" default="-1.57" />
   <!-- Farmily-specific links and joints belong below this line. -->
+  <link name="$(arg prefix)farmily_lift">
+    <visual>
+      <geometry>
+        <!-- Assy_Lift.STL is authored in millimetres. -->
+        <mesh
+          filename="package://rbpodo_description/meshes/farmily_lift/assy_lift.stl"
+          scale="0.001 0.001 0.001" />
+      </geometry>
+      <material name="farmily_lift_gray">
+        <color rgba="0.32 0.34 0.38 1.0" />
+      </material>
+    </visual>
+  </link>
+  <joint name="$(arg prefix)farmily_lift_joint" type="fixed">
+    <origin
+      xyz="$(arg lift_mount_x) $(arg lift_mount_y) $(arg lift_mount_z)"
+      rpy="$(arg lift_mount_roll) $(arg lift_mount_pitch) $(arg lift_mount_yaw)" />
+    <parent link="$(arg prefix)link0" />
+    <child link="$(arg prefix)farmily_lift" />
+  </joint>
   <link name="$(arg prefix)tomato_gripper">
     <visual>

Commit message: RViz 리프트 승강 모델과 시뮬레이션 제어 추가
회색 리프트 프레임은 world에 고정하고 초록색 승강판과 link0 이하 RB5 전체가 prismatic lift joint를 따라 함께 이동하도록 rb5_farmily 모델을 재구성한다.

실제 리프트의 Bottom 기준 높이를 mm에서 m로 변환해 joint_states에 공급하는 브리지 노드를 추가하고 MoveIt에서 lift joint를 passive joint로 관리한다. 다른 로봇 모델에는 기존 static world-link0 TF를 유지한다.

fake hardware에서는 실제 lift_control 토픽과 분리된 lift_simulation 토픽만 사용해 GUI 높이 조정이 RViz 모델에만 적용되도록 한다. 실제 모드에서는 기존 lift node, Bottom calibration 및 실측 높이를 계속 사용한다.

URDF 트리, MoveIt 기동, 실제 높이 TF 변환, simulation command isolation과 GUI 동작을 테스트한다.

File: ros2_ws/src/rbpodo_ros2/rbpodo_description/robots/rb5_farmily.urdf.xacro (robot description, xacro)
@@ -10,5 +10,5 @@
   <xacro:arg name="d435_mount_pitch" default="0.0" />
   <xacro:arg name="d435_mount_yaw" default="3.141592" />
-  <!-- Farmily lift pose relative to the RB5 base frame (link0). -->
+  <!-- Farmily lift pose in the stationary world frame. -->
   <xacro:arg name="lift_mount_x" default="0.0" />
   <xacro:arg name="lift_mount_y" default="0.6" />
@@ -17,4 +17,14 @@
   <xacro:arg name="lift_mount_pitch" default="0.0" />
   <xacro:arg name="lift_mount_yaw" default="-1.57" />
+  <!-- Moving green platform. Its link frame stays directly below link0. -->
+  <xacro:arg name="lift_platform_size_x" default="0.30" />
+  <xacro:arg name="lift_platform_size_y" default="0.95" />
+  <xacro:arg name="lift_platform_thickness" default="0.025" />
+  <xacro:arg name="lift_platform_visual_x" default="0.0" />
+  <xacro:arg name="lift_platform_visual_y" default="0.30" />
+  <xacro:arg name="lift_min_height" default="0.0" />
+  <xacro:arg name="lift_max_height" default="1.20" />
+  <!-- The model is rooted in world so the lift can move the complete RB5. -->
+  <link name="world" />
   <!-- Farmily-specific links and joints belong below this line. -->
   <link name="$(arg prefix)farmily_lift">
@@ -31,10 +41,50 @@
     </visual>
   </link>
-  <joint name="$(arg prefix)farmily_lift_joint" type="fixed">
+  <joint name="$(arg prefix)farmily_lift_fixed_joint" type="fixed">
     <origin
       xyz="$(arg lift_mount_x) $(arg lift_mount_y) $(arg lift_mount_z)"
       rpy="$(arg lift_mount_roll) $(arg lift_mount_pitch) $(arg lift_mount_yaw)" />
-    <parent link="$(arg prefix)link0" />
+    <parent link="world" />
     <child link="$(arg prefix)farmily_lift" />
+  </joint>
+  <link name="$(arg prefix)farmily_lift_platform">
+    <visual>
+      <origin
+        xyz="$(arg lift_platform_visual_x) $(arg lift_platform_visual_y) 0"
+        rpy="0 0 0" />
+      <geometry>
+        <box
+          size="$(arg lift_platform_size_x) $(arg lift_platform_size_y) $(arg lift_platform_thickness)" />
+      </geometry>
+      <material name="farmily_lift_platform_green">
+        <color rgba="0.12 0.68 0.06 1.0" />
+      </material>
+    </visual>
+    <collision>
+      <origin
+        xyz="$(arg lift_platform_visual_x) $(arg lift_platform_visual_y) 0"
+        rpy="0 0 0" />
+      <geometry>
+        <box
+          size="$(arg lift_platform_size_x) $(arg lift_platform_size_y) $(arg lift_platform_thickness)" />
+      </geometry>
+    </collision>
+  </link>
+  <!-- The joint value is the physical Bottom-relative lift height in metres. -->
+  <joint name="$(arg prefix)farmily_lift_height_joint" type="prismatic">
+    <origin xyz="0 0 ${-0.5 * float($(arg lift_platform_thickness))}" rpy="0 0 0" />
+    <parent link="world" />
+    <child link="$(arg prefix)farmily_lift_platform" />
+    <axis xyz="0 0 1" />
+    <limit
+      lower="$(arg lift_min_height)"
+      upper="$(arg lift_max_height)"
+      effort="2000.0"
+      velocity="0.25" />
+  </joint>
+  <joint name="$(arg prefix)farmily_lift_robot_mount_joint" type="fixed">
+    <origin xyz="0 0 ${0.5 * float($(arg lift_platform_thickness))}" rpy="0 0 0" />
+    <parent link="$(arg prefix)farmily_lift_platform" />
+    <child link="$(arg prefix)link0" />
   </joint>
   <link name="$(arg prefix)tomato_gripper">

Commit message: 카메라 검출 시각화와 단계별 수확 실행 기능 추가
- Fake/실제 카메라 검출 소스를 GUI에서 선택하고 실제 서비스 응답을 토마토 검출 토픽으로 연계

- 검출 중심·줄기점·예상 진입 방향과 실제 계획 진입 방향을 RViz 마커로 표시하고 마커 크기 및 유지 동작 개선

- 카메라 optical frame 호환 TF와 RViz Camera display 설정을 MoveIt 실행 구성에 추가

- 전체 수확 trajectory를 10개 단계로 캐시하고 다음 단계 또는 선택 단계까지 실제 실행하는 전용 스텝 세션 구현

- 단계 실행 직전 실제 관절 시작 오차를 검증하고 실패 캐시 재사용 차단 및 즉시 정지 연동

- 그리퍼 visual/collision mesh를 Assy_4 모델로 교체하고 관련 문서와 단위 테스트 보강

File: ros2_ws/src/rbpodo_ros2/rbpodo_description/robots/rb5_farmily.urdf.xacro (robot description, xacro)
@@ -4,6 +4,6 @@
   <xacro:include filename="$(find rbpodo_description)/robots/rb5_850e.urdf.xacro" />
   <xacro:include filename="$(find rbpodo_description)/robots/realsense_d435.urdf.xacro" />
-  <xacro:arg name="d435_mount_x" default="-0.11" />
-  <xacro:arg name="d435_mount_y" default="-0.10" />
+  <xacro:arg name="d435_mount_x" default="-0.076" />
+  <xacro:arg name="d435_mount_y" default="-0.161" />
   <xacro:arg name="d435_mount_z" default="0.0" />
   <xacro:arg name="d435_mount_roll" default="-1.57" />
@@ -93,5 +93,5 @@
         <!-- The CAD mesh is authored in millimetres. -->
         <mesh
-          filename="package://rbpodo_description/meshes/tomato_gripper/assy_gripper_ver_4.stl"
+          filename="package://rbpodo_description/meshes/tomato_gripper/assy_4.stl"
           scale="0.001 0.001 0.001" />
       </geometry>
@@ -103,5 +103,5 @@
       <geometry>
         <mesh
-          filename="package://rbpodo_description/meshes/tomato_gripper/assy_gripper_ver_4.stl"
+          filename="package://rbpodo_description/meshes/tomato_gripper/assy_4.stl"
           scale="0.001 0.001 0.001" />
       </geometry>
@@ -120,5 +120,5 @@
   <link name="$(arg prefix)tomato_gripper_tip" />
   <joint name="$(arg prefix)tomato_gripper_tip_joint" type="fixed">
-    <origin xyz="-0.2116 0.01075 0" rpy="1.57 3.14 0" />
+    <origin xyz="-0.1816 0.01075 0" rpy="1.57 3.14 0" />
     <parent link="$(arg prefix)tomato_gripper" />
     <child link="$(arg prefix)tomato_gripper_tip" />

Commit message: 수확 단계 커스텀 설정과 비전 피드백 뷰어를 개선
- Assy Gripper Ver.5 메시를 로봇 visual/collision 모델에 적용하고 카메라 장착 위치 및 RViz 표시 설정을 갱신
- 수확 4단계 진입 길이와 스텝 3~7단계 tip 로컬 XYZ 이동량을 GUI에서 조정하도록 확장
- 변경된 전진·상승 수확 시퀀스를 개별, 반복, 전체 수확 경로에 일관되게 반영
- 검출 순간의 토마토 및 줄기점을 link0 좌표로 보존해 비전 피드백 JSON의 좌표 왜곡을 제거
- 측면 뷰어에서 실제 좌표 비율, 줄기점 가시성, 마커 테두리와 범례 배치를 개선
- RViz 검출 벡터 기반 Recommend 화살표와 Planner 최종 보정 화살표를 분리해 진입각을 정확히 비교
- 관련 단위 테스트와 사용 문서를 보강

File: ros2_ws/src/rbpodo_ros2/rbpodo_description/robots/rb5_farmily.urdf.xacro (robot description, xacro)
@@ -5,5 +5,5 @@
   <xacro:include filename="$(find rbpodo_description)/robots/realsense_d435.urdf.xacro" />
   <xacro:arg name="d435_mount_x" default="-0.076" />
-  <xacro:arg name="d435_mount_y" default="-0.161" />
+  <xacro:arg name="d435_mount_y" default="-0.012" />
   <xacro:arg name="d435_mount_z" default="0.0" />
   <xacro:arg name="d435_mount_roll" default="-1.57" />
@@ -93,5 +93,5 @@
         <!-- The CAD mesh is authored in millimetres. -->
         <mesh
-          filename="package://rbpodo_description/meshes/tomato_gripper/assy_4.stl"
+          filename="package://rbpodo_description/meshes/tomato_gripper/assy_gripper_ver_5.stl"
           scale="0.001 0.001 0.001" />
       </geometry>
@@ -103,5 +103,5 @@
       <geometry>
         <mesh
-          filename="package://rbpodo_description/meshes/tomato_gripper/assy_4.stl"
+          filename="package://rbpodo_description/meshes/tomato_gripper/assy_gripper_ver_5.stl"
           scale="0.001 0.001 0.001" />
       </geometry>
@@ -120,5 +120,5 @@
   <link name="$(arg prefix)tomato_gripper_tip" />
   <joint name="$(arg prefix)tomato_gripper_tip_joint" type="fixed">
-    <origin xyz="-0.1816 0.01075 0" rpy="1.57 3.14 0" />
+    <origin xyz="-0.1816 0.01075 0" rpy="1.57 3.14 0.0" />
     <parent link="$(arg prefix)tomato_gripper" />
     <child link="$(arg prefix)tomato_gripper_tip" />

Commit message: 그리퍼 모델 교체 및 PIN10 서보 속도 제어 추가
토마토 그리퍼 visual/collision 메시를 Assy_Gripper_ver.3_ver2로 교체하고 표시 여부를 Xacro와 MoveIt 런치 인자로 제어하도록 구성했다. 기본값과 시뮬레이션·실제 로봇 실행 스크립트는 모두 그리퍼 표시로 설정했다.

GUI에 PIN10 서보 90도 닫기와 170도 열기 버튼을 추가하고 사용자 지정 속도 체크박스 및 1% 단위 Spinbox를 연결했다. 체크 해제 시 기본 50%(임시 기준 90deg/s), 체크 시 1~100% 사용자 값을 사용한다.

각도와 속도를 Float64MultiArray 단일 명령으로 전송하고 Arduino 브리지가 ANGLE 10 <angle> <speed> 직렬 명령으로 변환하도록 했다. 펌웨어에는 1~99% 비차단 각도 보간과 100% 즉시 이동을 추가했으며 관련 검증 테스트와 사용 문서를 갱신했다.

File: ros2_ws/src/rbpodo_ros2/rbpodo_description/robots/rb5_farmily.urdf.xacro (robot description, xacro)
@@ -4,6 +4,8 @@
   <xacro:include filename="$(find rbpodo_description)/robots/rb5_850e.urdf.xacro" />
   <xacro:include filename="$(find rbpodo_description)/robots/realsense_d435.urdf.xacro" />
-  <xacro:arg name="d435_mount_x" default="-0.076" />
-  <xacro:arg name="d435_mount_y" default="-0.006" />
+  <!-- Hide only the mesh in RViz; collision and TCP remain active. -->
+  <xacro:arg name="show_tomato_gripper" default="true" />
+  <xacro:arg name="d435_mount_x" default="-0.08435" />
+  <xacro:arg name="d435_mount_y" default="0.0859" />
   <xacro:arg name="d435_mount_z" default="0.0" />
   <xacro:arg name="d435_mount_roll" default="-1.57" />
@@ -89,19 +91,21 @@
   </joint>
   <link name="$(arg prefix)tomato_gripper">
-    <visual>
-      <geometry>
-        <!-- The CAD mesh is authored in millimetres. -->
-        <mesh
-          filename="package://rbpodo_description/meshes/tomato_gripper/assy_gripper_ver_5.stl"
-          scale="0.001 0.001 0.001" />
-      </geometry>
-      <material name="tomato_gripper_gray">
-        <color rgba="0.25 0.25 0.28 1.0" />
-      </material>
-    </visual>
+    <xacro:if value="$(arg show_tomato_gripper)">
+      <visual>
+        <geometry>
+          <!-- The CAD mesh is authored in millimetres. -->
+          <mesh
+            filename="package://rbpodo_description/meshes/tomato_gripper/assy_gripper_ver_3_ver2.stl"
+            scale="0.001 0.001 0.001" />
+        </geometry>
+        <material name="tomato_gripper_gray">
+          <color rgba="0.25 0.25 0.28 1.0" />
+        </material>
+      </visual>
+    </xacro:if>
     <collision>
       <geometry>
         <mesh
-          filename="package://rbpodo_description/meshes/tomato_gripper/assy_gripper_ver_5.stl"
+          filename="package://rbpodo_description/meshes/tomato_gripper/assy_gripper_ver_3_ver2.stl"
           scale="0.001 0.001 0.001" />
       </geometry>
@@ -120,5 +124,5 @@
   <link name="$(arg prefix)tomato_gripper_tip" />
   <joint name="$(arg prefix)tomato_gripper_tip_joint" type="fixed">
-    <origin xyz="-0.1816 0.01075 0" rpy="1.57 3.14 0.0" />
+    <origin xyz="-0.162 -0.006 0" rpy="1.57 3.14 0.0" />
     <parent link="$(arg prefix)tomato_gripper" />
     <child link="$(arg prefix)tomato_gripper_tip" />

Commit message: 수확 경로 안정화와 스텝 웨이브 옵션 추가
- READY와 PRE_APPROACH 사이에 작물 외곽 안전 경유점을 계산하고 복귀 경로에도 적용

- 스텝 4 전진 모션의 Z축 웨이브를 선택 옵션으로 분리하고 기본값을 비활성화

- 웨이브 사용 시 단일 Cartesian 경로로 검증하고 미사용 시 기존 직선 및 OMPL fallback 유지

- 스텝별 서보 닫기 각도와 리니어모터 3초 늘림/줄임 시퀀스를 GUI와 실행기에 연동

- 실측 관절 기준 trajectory 완료 판정과 정밀 named pose 목표 허용오차를 적용

- 관절 회전 범위 검증과 Cartesian 경로 안정성 테스트 및 GUI 옵션 회귀 테스트 보강

File: ros2_ws/src/rbpodo_ros2/rbpodo_description/robots/rb5_farmily.urdf.xacro (robot description, xacro)
@@ -124,5 +124,5 @@
   <link name="$(arg prefix)tomato_gripper_tip" />
   <joint name="$(arg prefix)tomato_gripper_tip_joint" type="fixed">
-    <origin xyz="-0.162 -0.006 0" rpy="1.57 3.14 0.0" />
+    <origin xyz="-0.162 0.020 0" rpy="1.57 3.14 0.0" />
     <parent link="$(arg prefix)tomato_gripper" />
     <child link="$(arg prefix)tomato_gripper_tip" />

Commit message: 스텝 수확 속도 제어와 액추에이터 시퀀스 개선
- 2단계 경유점 A 사용 여부와 A→PRE_APPROACH 속도를 GUI에서 선택하도록 추가

- 3~8단계와 복귀 이탈 구간의 속도를 개별 설정하고 캐시 궤적 재타이밍 및 전체 경로 병합을 지원

- PRE_APPROACH 계획 자세를 RViz Query Goal로 발행하는 디버깅 기능 추가

- 리니어모터 늘림 시간을 설정 가능하게 하고 서보 닫기/열기 각도 및 관련 문서를 현 하드웨어 값으로 갱신

- 서보 닫기 0.7초, 열기 0.7초 뒤 리니어모터 줄임을 비동기로 시작하고 3초 후 자동 LOW 처리

- RB Speed Bar를 자동 100%로 유지하며 단계별 계획 속도와 하드웨어 속도의 역할을 분리

- 신규 그리퍼 STL과 카메라 마운트 및 gripper tip 좌표를 로봇 모델에 반영

- 궤적 병합·속도 제한·서보·리니어모터 동작 회귀 테스트 보강

File: ros2_ws/src/rbpodo_ros2/rbpodo_description/robots/rb5_farmily.urdf.xacro (robot description, xacro)
@@ -6,7 +6,7 @@
   <!-- Hide only the mesh in RViz; collision and TCP remain active. -->
   <xacro:arg name="show_tomato_gripper" default="true" />
-  <xacro:arg name="d435_mount_x" default="-0.08435" />
-  <xacro:arg name="d435_mount_y" default="0.0859" />
-  <xacro:arg name="d435_mount_z" default="0.0" />
+  <xacro:arg name="d435_mount_x" default="-0.04915" />
+  <xacro:arg name="d435_mount_y" default="0.0415" />
+  <xacro:arg name="d435_mount_z" default="0.0125" />
   <xacro:arg name="d435_mount_roll" default="-1.57" />
   <xacro:arg name="d435_mount_pitch" default="0.0" />
@@ -96,5 +96,5 @@
           <!-- The CAD mesh is authored in millimetres. -->
           <mesh
-            filename="package://rbpodo_description/meshes/tomato_gripper/assy_gripper_ver_3_ver2.stl"
+            filename="package://rbpodo_description/meshes/tomato_gripper/assy_gripper_ver_3_1.stl"
             scale="0.001 0.001 0.001" />
         </geometry>
@@ -107,5 +107,5 @@
       <geometry>
         <mesh
-          filename="package://rbpodo_description/meshes/tomato_gripper/assy_gripper_ver_3_ver2.stl"
+          filename="package://rbpodo_description/meshes/tomato_gripper/assy_gripper_ver_3_1.stl"
           scale="0.001 0.001 0.001" />
       </geometry>
@@ -124,5 +124,5 @@
   <link name="$(arg prefix)tomato_gripper_tip" />
   <joint name="$(arg prefix)tomato_gripper_tip_joint" type="fixed">
-    <origin xyz="-0.162 0.020 0" rpy="1.57 3.14 0.0" />
+    <origin xyz="-0.133 0.006 0" rpy="1.57 3.14 0.0" />
     <parent link="$(arg prefix)tomato_gripper" />
     <child link="$(arg prefix)tomato_gripper_tip" />
